File: sd_mux/sd_mux.sch (KiCad schematic (older format))
At the start: 16 parts, among them IC1 SN74CBT3257DR, IC2 SN74CBT3257DR, J1 Micro_SD_Card_Det, J2 DEVICE 1, J3 DEVICE 2, J4 CONTROL

Commit message: Use the SN74CB3Q3257.
Parts:
- C1, C2, C3: symbol C_Small -> sd_mux-rescue:C_Small
- IC1, IC2: symbol SN74CBT3257DR -> sd_mux_library:SN74CBT3257DR
- J1: symbol Micro_SD_Card_Det -> sd_mux-rescue:Micro_SD_Card_Det
- J2, J3: symbol Conn_01x12 -> sd_mux-rescue:Conn_01x12
- J4: symbol Conn_01x03 -> sd_mux-rescue:Conn_01x03
- LED1, LED2: symbol LED -> sd_mux-rescue:LED
- R1, R2, R3, R4, R5: symbol R -> sd_mux-rescue:R
Connections:
- wire segments 122 -> 144
Changed lines of the file:
@@
-EESchema Schematic File Version 2
-LIBS:sd_mux-rescue
-LIBS:power
-LIBS:device
-LIBS:transistors
-LIBS:conn
-LIBS:linear
-LIBS:regul
-LIBS:74xx
-LIBS:cmos4000
-LIBS:adc-dac
-LIBS:memory
-LIBS:xilinx
-LIBS:microcontrollers
-LIBS:dsp
-LIBS:microchip
-LIBS:analog_switches
-LIBS:motorola
-LIBS:texas
-LIBS:intel
-LIBS:audio
-LIBS:interface
-LIBS:digital-audio
-LIBS:philips
-LIBS:display
-LIBS:cypress
-LIBS:siliconi
-LIBS:opto
-LIBS:atmel
-LIBS:contrib
-LIBS:valves
-LIBS:sd_mux_library
-LIBS:sd_mux-cache
-EELAYER 25 0
+EESchema Schematic File Version 4
+EELAYER 30 0
 EELAYER END
 $Descr A4 11693 8268
@@
 $EndDescr
 $Comp
-L Micro_SD_Card_Det J1
+L sd_mux-rescue:Micro_SD_Card_Det J1
 U 1 1 5A0DE1ED
 P 8300 3400
@@
 $EndComp
 $Comp
-L SN74CBT3257DR IC1
+L sd_mux_library:SN74CBT3257DR IC1
 U 1 1 5A0DDE4F
 P 5450 2400
@@
 $EndComp
 $Comp
-L SN74CBT3257DR IC2
+L sd_mux_library:SN74CBT3257DR IC2
 U 1 1 5A0DDEBA
 P 5450 4000
@@
 $EndComp
 $Comp
-L Conn_01x12 J2
+L sd_mux-rescue:Conn_01x12 J2
 U 1 1 5A0DE162
 P 2250 2350
@@
 $EndComp
 $Comp
-L Conn_01x12 J3
+L sd_mux-rescue:Conn_01x12 J3
 U 1 1 5A0DE319
 P 2250 3950
@@
 $EndComp
 $Comp
-L GND #PWR01
+L power1:GND #PWR01
 U 1 1 5A0DE7CC
 P 6350 2900
@@
 $EndComp
 $Comp
-L GND #PWR02
+L power1:GND #PWR02
 U 1 1 5A0DE82E
 P 6550 5000
@@
 $EndComp
 $Comp
-L GND #PWR03
+L power1:GND #PWR03
 U 1 1 5A0DE90A
 P 8050 5850
@@
 $EndComp
 $Comp
-L GND #PWR04
+L power1:GND #PWR04
 U 1 1 5A0DEA23
 P 7300 4050
@@
 $EndComp
 $Comp
-L GND #PWR05
+L power1:GND #PWR05
 U 1 1 5A0DEA83
 P 9250 3900
@@
 $EndComp
 $Comp
-L VCC #PWR06
+L power1:VCC #PWR06
 U 1 1 5A0DECC1
 P 6550 3600
@@
 $EndComp
 $Comp
-L VCC #PWR07
+L power1:VCC #PWR07
 U 1 1 5A0DED29
 P 6350 1950
@@
 $EndComp
 $Comp
-L VCC #PWR08
+L power1:VCC #PWR08
 U 1 1 5A0DEDB5
 P 8150 5250
@@
 device_select
 $Comp
-L Conn_01x03 J4
+L sd_mux-rescue:Conn_01x03 J4
 U 1 1 5A0DFB80
 P 8350 5750
@@
 device_select
 $Comp
-L R R1
+L sd_mux-rescue:R R1
 U 1 1 5A0E00B7
 P 7900 5550
@@
 OE
 $Comp
-L R R2
+L sd_mux-rescue:R R2
 U 1 1 5A0E043C
 P 5750 4950
@@
 DAT1_2
 $Comp
-L GND #PWR09
+L power1:GND #PWR09
 U 1 1 5A0E48B7
 P 2600 4750
@@
 $EndComp
 $Comp
-L VCC #PWR010
+L power1:VCC #PWR010
 U 1 1 5A0E5053
 P 7650 4900
@@
 $EndComp
 $Comp
-L R R3
+L sd_mux-rescue:R R3
 U 1 1 5A0E566E
 P 6950 5000
@@
 $EndComp
 $Comp
-L R R4
+L sd_mux-rescue:R R4
 U 1 1 5A0E570C
 P 6950 5300
@@
 $EndComp
 $Comp
-L GND #PWR011
+L power1:GND #PWR011
 U 1 1 5A0E5B3E
 P 6700 5400
@@
 $EndComp
 $Comp
-L C_Small C1
+L sd_mux-rescue:C_Small C1
 U 1 1 5A0E0A40
 P 6350 2100
@@
 $EndComp
 $Comp
-L C_Small C2
+L sd_mux-rescue:C_Small C2
 U 1 1 5A0E1230
 P 6550 3700
@@
 $EndComp
 $Comp
-L C_Small C3
+L sd_mux-rescue:C_Small C3
 U 1 1 5A0E19BB
 P 6800 3400
@@
 $EndComp
 $Comp
-L PWR_FLAG #FLG012
+L power1:PWR_FLAG #FLG012
 U 1 1 5A0EEB4C
 P 2500 6250
@@
 $EndComp
 $Comp
-L PWR_FLAG #FLG013
+L power1:PWR_FLAG #FLG013
 U 1 1 5A0EEB7E
 P 2900 6250
@@
 $EndComp
 $Comp
-L GND #PWR014
+L power1:GND #PWR014
 U 1 1 5A0EEBB0
 P 2500 6350
@@
 $EndComp
 $Comp
-L VCC #PWR015
+L power1:VCC #PWR015
 U 1 1 5A0EEBE2
 P 2900 6350
@@
 $EndComp
 $Comp
-L LED LED1
+L sd_mux-rescue:LED LED1
 U 1 1 5A0F157B
 P 7350 5000
@@
 $EndComp
 $Comp
-L LED LED2
+L sd_mux-rescue:LED LED2
 U 1 1 5A0F15B8
 P 7350 5300
@@
 NoConn ~ 4700 4200
 $Comp
-L R R5
+L sd_mux-rescue:R R5
 U 1 1 5A0F2C39
 P 6300 4650
@@
 $EndComp
 $Comp
-L PWR_FLAG #FLG016
+L power1:PWR_FLAG #FLG016
 U 1 1 5A0F446F
 P 6600 3300
@@
 	6150 2850 6350 2850
 Wire Wire Line
-	6350 2200 6350 2900
+	6350 2200 6350 2850
 Wire Wire Line
 	6550 4450 6150 4450
 Wire Wire Line
-	6800 3500 7400 3500
+	6800 3500 7300 3500
 Wire Wire Line
 	9250 3900 9100 3900
@@
 	7050 2450 6150 2450
 Wire Wire Line
-	6600 3300 7400 3300
+	6600 3300 6800 3300
 Wire Wire Line
 	6950 3300 6950 2550
@@
 	7150 3700 7150 4150
 Wire Wire Line
-	6550 3800 6550 5000
-Wire Wire Line
-	7300 3500 7300 4050
+	6550 3800 6550 4450
+Wire Wire Line
+	7300 3500 7300 3800
 Wire Wire Line
 	7400 3800 7300 3800
@@
 	5400 4700 5250 4700
 Wire Wire Line
-	7350 5750 8150 5750
+	7350 5750 7650 5750
 Connection ~ 7900 5750
 Wire Wire Line
 	5650 3100 5500 3100
 Wire Wire Line
-	5500 4700 5650 4700
+	5500 4700 5550 4700
 Wire Wire Line
 	5550 4700 5550 4950
@@
 Connection ~ 6550 4450
 Wire Wire Line
-	5900 4950 6550 4950
+	5900 4950 6300 4950
 Connection ~ 6550 4950
 Connection ~ 7300 3900
@@
 	8150 5850 8050 5850
 Wire Wire Line
-	8150 5250 8150 5650
+	8150 5250 8150 5300
 Connection ~ 8150 5300
 Wire Wire Line
@@
 	7200 5300 7100 5300
 Wire Wire Line
-	6700 5000 6700 5400
+	6700 5000 6700 5300
 Wire Wire Line
 	6700 5000 6800 5000
@@
 Wire Wire Line
 	6300 3950 6300 4500
-Wire Wire Line
-	6800 3300 6800 3300
 Connection ~ 6800 3300
 Wire Wire Line
@@
 	2500 2400 2700 2400
 Wire Wire Line
-	2600 1950 2600 4750
+	2600 1950 2600 2150
 Wire Wire Line
 	2450 3450 2800 3450
@@
 	2450 3550 2600 3550
 Connection ~ 2600 3550
+Wire Wire Line
+	7300 3800 7300 3900
+Wire Wire Line
+	7900 5750 8150 5750
+Wire Wire Line
+	5550 4700 5650 4700
+Wire Wire Line
+	6550 4450 6550 4950
+Wire Wire Line
+	6550 4950 6550 5000
+Wire Wire Line
+	7300 3900 7300 4050
+Wire Wire Line
+	8150 5300 8150 5650
+Wire Wire Line
+	6700 5300 6700 5400
+Wire Wire Line
+	7650 5750 7900 5750
+Wire Wire Line
+	6350 2850 6350 2900
+Wire Wire Line
+	6950 3300 7400 3300
+Wire Wire Line
+	7300 3500 7400 3500
+Wire Wire Line
+	6300 4950 6550 4950
+Wire Wire Line
+	6800 3300 6950 3300
+Wire Wire Line
+	2600 2150 2600 2350
+Wire Wire Line
+	2600 2350 2600 2650
+Wire Wire Line
+	2600 2650 2600 2850
+Wire Wire Line
+	2600 2850 2600 3550
+Wire Wire Line
+	2600 4450 2600 4750
+Wire Wire Line
+	2600 3950 2600 4250
+Wire Wire Line
+	2600 4250 2600 4450
+Wire Wire Line
+	2600 3750 2600 3950
+Wire Wire Line
+	2600 3550 2600 3750
 $EndSCHEMATC
